File: KiCad/ESP LoRa Schematic/_autosave-ESP LoRa Schematic.kicad_sch (KiCad schematic)
At the start: 11 parts, among them J1 Conn_01x05_Socket, J2 Conn_01x02_Socket, J3 Conn_01x07_Socket, U1 ESP32-S3-DEVKITC-1-N8R8, U2 RA-02_LORA

Commit message: add feature
add second UART line for configureing UART
Parts:
- H1, H2, H3, H4: footprint MountingHole:MountingHole_4.3mm_M4_DIN965_Pad -> MountingHole:MountingHole_3.2mm_M3_ISO14580_Pad
Connections:
- net +3.3V: now also OLED1.2 (Pin_2); no longer OLED1.4 (Pin_4)
- net GND: now also OLED1.1 (Pin_1); no longer OLED1.3 (Pin_3)
- net GPIO17: now also U3.30 (PA3); no longer U3.6 (TX1)
- net GPIO18: now also U3.31 (PA2); no longer U3.7 (RX1)
- net GPIO8: now also OLED1.4 (Pin_4); no longer OLED1.1 (Pin_1)
- net GPIO9: now also OLED1.3 (Pin_3); no longer OLED1.2 (Pin_2)
- net GPIO6: now reaches U1.J1_6 (GPIO6)
- net GPIO6: now also U3.6 (TX1)
- net GPIO7: now reaches U1.J1_7 (GPIO7)
- net GPIO7: now also U3.7 (RX1)
- net GPIO15: now reaches U1.J1_8 (GPIO15)
- net GPIO15: now also U3.24 (NRST)
- net GPIO43: no longer names the net of U1.J3_2 (U0TXD/GPIO43)
- net GPIO43: no longer U3.31 (PA2)
- net GPIO44: no longer names the net of U1.J3_3 (U0RXD/GPIO44)
- net GPIO44: no longer U3.30 (PA3)
- no-connect marks 70 -> 67
Other:
- note added: "UWB RESET"
- note added: "UWB RX"
- note added: "UWB TX"
- moved on the sheet: J3, OLED1
