File: KiCad/Egg/Egg.kicad_pcb (KiCad board)
At the start: 4 copper layers, 90 x 60 mm, 20 parts, among them J1 Conn_01x05_Socket, J2 Conn_01x02_Socket, J3 Conn_01x07_Socket, J4 Conn_01x02_Socket, J5 Conn_01x02_Socket, J6 Conn_01x02_Socket, U1 ESP32-S3-DEVKITC-1-N8R8, U2 RA-02_LORA

Commit message: production pcb
Parts:
- removed OLED1: Conn_01x04_Socket, Connector_JST:JST_XH_B4B-XH-A_1x04_P2.50mm_Vertical
- added J7: Conn_01x05_Socket, Connector_JST:JST_XH_B5B-XH-A_1x05_P2.50mm_Vertical, F.Cu at (138.8, 120.2)
- added J8: Conn_01x04_Socket, Connector_JST:JST_XH_B4B-XH-A_1x04_P2.50mm_Vertical, B.Cu at (177.8, 92.9)
- J1: value Conn_01x05_Socket -> Conn_01x02_Socket; footprint Connector_JST:JST_XH_B5B-XH-A_1x05_P2.50mm_Vertical -> Connector_JST:JST_PH_B2B-PH-K_1x02_P2.00mm_Vertical
- J2: footprint Connector_JST:JST_PH_B2B-PH-K_1x02_P2.00mm_Vertical -> Connector_JST:JST_XH_B2B-XH-A_1x02_P2.50mm_Vertical
- J3: value Conn_01x07_Socket -> Conn_01x02_Socket; footprint Connector_JST:JST_XH_B7B-XH-A_1x07_P2.50mm_Vertical -> Connector_JST:JST_XH_B2B-XH-A_1x02_P2.50mm_Vertical
- J5: value Conn_01x02_Socket -> Conn_01x04_Socket; footprint Connector_JST:JST_XH_B2B-XH-A_1x02_P2.50mm_Vertical -> Connector_JST:JST_XH_B4B-XH-A_1x04_P2.50mm_Vertical
- J6: value Conn_01x02_Socket -> Conn_01x03_Socket; footprint Connector_JST:JST_XH_B2B-XH-A_1x02_P2.50mm_Vertical -> Connector_JST:JST_XH_B3B-XH-A_1x03_P2.50mm_Vertical
- moved kibuzzard-69BA529B 71.1 mm to (150.3, 77.3), turned to 180 degrees
- moved J5 64.4 mm to (103.0, 120.2)
- moved J3 55.5 mm to (131.4, 72.5)
- moved J1 55.0 mm to (102.5, 72.5)
- moved J6 48.1 mm to (122.2, 120.2)
- moved kibuzzard-69BA525D 18.3 mm to (177.2, 88.6), turned to 180 degrees
- moved J4 15.0 mm to (146.3, 72.5)
- moved J2 14.1 mm to (116.6, 72.5)
- moved G*** 6.40 mm to (156.2, 120.7)
- moved kibuzzard-69BA5F59 6.20 mm to (167.1, 120.8)
- moved H2 6.00 mm to (177.5, 72.8)
- moved H3 6.00 mm to (177.5, 120.8)
- moved U2 6.00 mm to (180.9, 84.2)
- moved kibuzzard-69B7B320 6.00 mm to (162.9, 80.3)
Connections:
- J1 pad 1: GPIO8 -> +5V
- J1 pad 2: GPIO9 -> GND
- J3 pad 1: unconnected-(J3-Pin_1-Pad1) -> +5V
- J3 pad 2: unconnected-(J3-Pin_2-Pad2) -> GND
- J4 pad 1: +5V -> +3.3V
- J5 pad 1: +3.3V -> GPIO35
- J5 pad 2: GND -> GPIO36
- J6 pad 2: GND -> +3.3V
- U1 pad J3_1: GND -> unconnected-(U1-GND-PadJ3_1)
- U1 pad J3_10: unconnected-(U1-GPIO38-PadJ3_10) -> GPIO38
- U1 pad J3_11: unconnected-(U1-GPIO37-PadJ3_11) -> GPIO37
- U1 pad J3_12: unconnected-(U1-GPIO36-PadJ3_12) -> GPIO36
- U1 pad J3_13: unconnected-(U1-GPIO35-PadJ3_13) -> GPIO35
- U3 pad 30: GPIO17 -> GPIO18
- U3 pad 31: GPIO18 -> GPIO17
Routing:
- net GPIO38: track 0.00 -> 51.1 mm
- net GPIO37: track 0.00 -> 47.5 mm
- net GPIO36: track 0.00 -> 41.2 mm
- net GPIO35: track 0.00 -> 37.5 mm
- net +3.3V: track 231.9 -> 261.1 mm
- net GPIO10: track 71.2 -> 77.3 mm
- net GPIO5: track 27.0 -> 33.0 mm
- net GPIO4: track 27.4 -> 33.4 mm
- net GPIO12: track 67.9 -> 73.9 mm
- net GPIO11: track 70.5 -> 76.5 mm
- net GPIO13: track 73.0 -> 79.0 mm
- net GPIO8: track 100.2 -> 96.5 mm
- net GPIO9: track 110.0 -> 107.2 mm
- net +5V: track 150.1 -> 152.3 mm
- net GPIO18: track 6.14 -> 5.09 mm
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Other:
- board size 90 x 60 mm -> 96 x 60 mm
- board text added: "IO35"
- board text added: "IO36"
- board text added: "IO37"
- board text added: "IO38"
