File: KiCad/Egg/Egg.kicad_sch (KiCad schematic)
At the start: 14 parts, among them J1 Conn_01x05_Socket, J2 Conn_01x02_Socket, J3 Conn_01x07_Socket, J4 Conn_01x02_Socket, J5 Conn_01x02_Socket, J6 Conn_01x02_Socket, U1 ESP32-S3-DEVKITC-1-N8R8, U2 RA-02_LORA

Commit message: production pcb
Parts:
- removed J3: Conn_01x07_Socket, Connector_JST:JST_XH_B7B-XH-A_1x07_P2.50mm_Vertical, symbol Connector:Conn_01x07_Socket
- added J5: Conn_01x04_Socket, Connector_JST:JST_XH_B4B-XH-A_1x04_P2.50mm_Vertical, symbol Connector:Conn_01x04_Socket
- added J6: Conn_01x03_Socket, Connector_JST:JST_XH_B3B-XH-A_1x03_P2.50mm_Vertical, symbol Connector:Conn_01x03_Socket
- renumbered J2 to J1, J6 to J2, J4 to J3, J5 to J4, J1 to J7, OLED1 to J8
Connections:
- net +3.3V: now also J6.2 (Pin_2)
- net +5V: now also J7.3 (Pin_3), J6.1 (Pin_1); no longer J7.5 (Pin_5)
- net GND: now also J7.5 (Pin_5), J6.3 (Pin_3); no longer J7.3 (Pin_3), U1.J3_1 (GND)
- net GPIO17: now also U3.31 (PA2); no longer U3.30 (PA3)
- net GPIO18: now also U3.30 (PA3); no longer U3.31 (PA2)
- net GPIO38: now reaches U1.J3_10 (GPIO38)
- net GPIO38: now also J5.4 (Pin_4)
- net GPIO37: now reaches U1.J3_11 (GPIO37)
- net GPIO37: now also J5.3 (Pin_3)
- net GPIO36: now reaches U1.J3_12 (GPIO36)
- net GPIO36: now also J5.2 (Pin_2)
- net GPIO35: now reaches U1.J3_13 (GPIO35)
- net GPIO35: now also J5.1 (Pin_1)
- no-connect marks 65 -> 61
Other:
- note removed: "SPI"
- moved on the sheet: H1, H2, H3, H4, J3, J4, J7, U1
